File: rtu-old/eagle/rtu.brd (EAGLE design)
At the start: 76.2 x 65.4 mm, 115 parts

Commit message: do
Parts:
- removed BAT1: (no value), myparts:BAT-1220-BC501SM
- removed C291, C301, C331: (no value), myparts:0603
- added C29, C30: (no value), myparts:0603
- C10, C14, R27, R32: device myparts:1206 -> myparts:0603
- C12, C9, R25: device myparts:0603 -> myparts:1206
- IC8: device myparts:SOIC-8 -> myparts:SOIC-8-208
- R16, R18, R36, R37: device myparts:0603 -> myparts:0805
- R21: device myparts:0805 -> myparts:1206
- R23, R41, R42: device myparts:0805 -> myparts:0603
- moved IC8 62.7 mm to (14.9, 37.5)
- moved R46 57.5 mm to (14.9, 42.9), turned to 180 degrees
- moved R47 55.7 mm to (14.9, 41.4), turned to 180 degrees
- moved R30 54.3 mm to (46.2, 28.8), turned to 270 degrees
- moved R7 52.7 mm to (59.8, 38.0), turned to 180 degrees
- moved R8 52.0 mm to (56.9, 36.4), turned to 0 degrees
- moved R18 48.1 mm to (21.5, 9.53), turned to 180 degrees
- moved C15 42.1 mm to (48.1, 38.0)
- moved R44 41.9 mm to (21.3, 45.8), turned to 180 degrees
- moved C18 40.2 mm to (17.0, 20.6)
- moved R45 39.9 mm to (21.3, 44.3), turned to 180 degrees
- moved R6 39.3 mm to (59.8, 36.4), turned to 0 degrees
- moved R25 36.7 mm to (38.5, 9.53), turned to 180 degrees
- moved R12 35.6 mm to (21.3, 36.7), turned to 0 degrees
- moved R5 34.3 mm to (10.3, 13.3), turned to 90 degrees
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- renumbered C34 to C31, C35 to C32
Connections:
- removed net N$23: IC5.3, R16.1, R25.2
- removed net N$81: CON5.5, R27.1, R28.2
- new net N$64: CON5.5, R21.1, R22.2
- new net N$86: IC1.41, R46.1
- new net N$87: IC8.2, R14.1
- net GND: now also C12.1, C23.1, C26.1, C28.2, C29.2, C30.2, C8.1, IC8.4, R32.1, R35.1, R42.1, R5.1; no longer BAT1.-, C10.1, C22.1, C25.1, C28.1, C291.1, C301.1, C331.1, C8.2, IC8.5, R37.1, R47.1, R6.1, R8.1
- net N$1: now also IC1.40, R44.1; no longer IC1.41, R5.1
- net N$13: now also C15.2, R11.2, R7.2, R9.2; no longer C17.2, R10.2, R12.2, R14.2
- net N$14: now also R6.1; no longer R9.1
- net N$15: now also R44.2; no longer R5.2
- net N$16: now also R8.1; no longer R11.1
- net N$17: now also C25.1, R26.2; no longer C26.1, R33.2
- net N$18: now also R2.1; no longer R1.1
- net N$19: now also R3.1; no longer R2.1
- net N$2: now also C17.2, R10.1, R11.1; no longer C18.2, R13.1, R14.1
- net N$20: now also R16.2; no longer R21.2
- net N$21: now also C25.2, R24.2; no longer C26.2, R31.2
- net N$22: now also R10.2; no longer R13.2
- net N$24: now also R41.2; no longer R46.2
- net N$25: now also IC8.1, R46.2, R47.2; no longer IC6.3, R17.1, R30.2
- net N$26: now also R41.1, R42.2; no longer R46.1, R47.2
- net N$27: now also R27.2; no longer R34.2
- net N$29: now also C28.1, R43.1; no longer C8.1, R4.1
- net N$3: now also R14.2, R15.2; no longer R17.2
- net N$30: now also R24.1, R25.1; no longer R31.1, R32.1
- net N$32: now also C19.2, R19.2; no longer C20.2, R24.2
- net N$33: now also R18.2; no longer R23.2
- net N$35: now also C18.2, R17.2; no longer C19.2, R22.2
- net N$36: now also R39.1, R40.2; no longer R44.1, R45.2
- net N$38: now also R39.2; no longer R44.2
- net N$40: now also R25.2, R26.1; no longer R32.2, R33.1
- net N$41: now also R1.2; no longer R3.2
- net N$42: now also C23.2; no longer C25.2
- net N$43: now also R2.2; no longer R1.2
- net N$44: now also R3.2; no longer R2.2
- net N$45: now also R12.2; no longer R15.2
- net N$47: now also R30.2, R31.2; no longer R35.2, R36.2
- net N$48: now also R34.2; no longer R39.2
- net N$51: now also R35.2, R36.2; no longer R40.2, R41.2
- net N$52: now also R37.2, R38.2; no longer R42.2, R43.2
- net N$53: now also R32.2, R33.2; no longer R37.2, R38.2
- net N$54: now also R37.1; no longer R42.1
- net N$55: now also R18.1; no longer R23.1
- net N$57: now also C9.2; no longer C10.2
- net N$58: now also R12.1; no longer BAT1.+, C291.2
- net N$59: now also R20.2, R21.2; no longer R26.2, R27.2
- net N$6: now also R6.2, R7.1; no longer R10.1, R9.2
- net N$61: now also R31.1; no longer R36.1
- net N$62: now also R34.1; no longer R39.1
- net N$63: now also R33.1; no longer R38.1
- net N$65: now also C11.2; no longer C12.2
- net N$66: now also C11.1; no longer C12.1
- net N$68: now also C22.2, R20.1; no longer C23.2, R26.1
- net N$69: now also C22.1, R22.1; no longer C23.1, R28.1
- net N$7: now also R8.2, R9.1; no longer R11.2, R12.1
- net N$70: now also IC8.5, R13.1; no longer IC8.3, R15.1, R18.2
- net N$71: now also R23.2; no longer R29.2
- net N$72: now also C10.1, R4.2, R5.2; no longer C11.1, R7.2, R8.2
- net N$73: now also R29.2; no longer IC8.8, R20.2
- net N$77: now also C20.2; no longer C22.2
- net N$79: now also R28.2; no longer IC8.7, R19.2
- net N$8: now also R45.2; no longer R6.2
- net N$80: now also R36.1; no longer R41.1
- net N$85: now also R16.1; no longer R21.1
- net N$9: now also R13.2; no longer R16.2
- net UVCC: now also C8.2; no longer C9.2
- net VCC: now also C10.2, C12.2, C26.2, C29.1, C30.1, IC8.3, IC8.7, IC8.8, R1.1, R15.1, R17.1, R23.1, R27.1, R28.1, R38.1, R4.1, R43.2, R47.1; no longer C11.2, C15.2, C28.2, C301.2, C331.2, IC8.2, R18.1, R20.1, R22.1, R24.1, R25.1, R3.1, R34.1, R35.1, R4.2, R43.1, R7.1
Routing:
- net VCC: track 241.7 -> 271.4 mm, vias 28 -> 31
- net N$86: track 0.00 -> 22.2 mm, vias 0 -> 2
- net N$87: track 0.00 -> 10.5 mm
- net N$3: track 6.81 -> 16.1 mm, vias 0 -> 1
- net N$9: track 11.8 -> 18.3 mm
- net N$25: track 0.00 -> 6.13 mm
- net GND: track 72.5 -> 76.6 mm, vias 62 -> 64
- net N$64: track 0.00 -> 3.68 mm
- net N$45: track 10.1 -> 13.5 mm
- net N$70: track 0.00 -> 2.32 mm
- net N$58: track 0.00 -> 2.21 mm
- net N$81: track 2.15 -> 0.00 mm
