File: rtu-old/eagle/rtu.sch (EAGLE design)
At the start: 115 parts

Commit message: do
Parts:
- removed BAT1: (no value), myparts:BAT-1220-BC501SM
- removed C221, C33: (no value), myparts:CAPACITOR-0603
- added C28: (no value), myparts:CAPACITOR-0603
- C10, C14: device myparts:CAPACITOR-1206 -> myparts:CAPACITOR-0603
- C12, C9: device myparts:CAPACITOR-0603 -> myparts:CAPACITOR-1206
- IC8: device myparts:DS3231M -> myparts:MEM-SPI-SOIC-8-208
- R16, R18, R36, R37: device myparts:RESISTOR-0603 -> myparts:RESISTOR-0805
- R21: device myparts:RESISTOR-0805 -> myparts:RESISTOR-1206
- R23, R41, R42: device myparts:RESISTOR-0805 -> myparts:RESISTOR-0603
- R25: device myparts:RESISTOR-0603 -> myparts:RESISTOR-1206
- R27, R32: device myparts:RESISTOR-1206 -> myparts:RESISTOR-0603
- renumbered C231 to C23, C241 to C24, C256 to C25, C261 to C26, C271 to C27
Connections:
- removed net N$23: IC5.ALR, R16.1, R25.2
- removed net N$81: CON5.5, R27.1, R28.2
- new net N$64: CON5.5, R21.1, R22.2
- new net N$86: IC1.ADC0/PF0, R46.1
- new net N$87: IC8.DO, R14.1
- net GND: now also C12.1, C28.2, C29.2, C30.2, C8.1, R32.1, R35.1, R42.1, R5.1; no longer BAT1.-, C10.1, C22.1, C29.1, C30.1, C33.1, C8.2, R37.1, R47.1, R6.1, R8.1
- net N$1: now also IC1.ADC1/PF1, R44.1; no longer IC1.ADC0/PF0, R5.1
- net N$13: now also C15.2, R11.2, R7.2, R9.2; no longer C17.2, R10.2, R12.2, R14.2
- net N$14: now also R6.1; no longer R9.1
- net N$15: now also R44.2; no longer R5.2
- net N$16: now also R8.1; no longer R11.1
- net N$17: now also R26.2; no longer R33.2
- net N$18: now also R2.1; no longer R1.1
- net N$19: now also R3.1; no longer R2.1
- net N$2: now also C17.2, R10.1, R11.1; no longer C18.2, R13.1, R14.1
- net N$20: now also R16.2; no longer R21.2
- net N$21: now also R24.2; no longer R31.2
- net N$22: now also R10.2; no longer R13.2
- net N$24: now also R41.2; no longer R46.2
- net N$25: now also IC8.!CS, R46.2, R47.2; no longer IC6.ALR, R17.1, R30.2
- net N$26: now also R41.1, R42.2; no longer R46.1, R47.2
- net N$27: now also R27.2; no longer R34.2
- net N$29: now also C28.1, R43.1; no longer C8.1, R4.1
- net N$3: now also R14.2, R15.2; no longer R17.2
- net N$30: now also R24.1, R25.1; no longer R31.1, R32.1
- net N$32: now also C19.2, R19.2; no longer C20.2, R24.2
- net N$33: now also R18.2; no longer R23.2
- net N$35: now also C18.2, R17.2; no longer C19.2, R22.2
- net N$36: now also R39.1, R40.2; no longer R44.1, R45.2
- net N$38: now also R39.2; no longer R44.2
- net N$40: now also R25.2, R26.1; no longer R32.2, R33.1
- net N$41: now also R1.2; no longer R3.2
- net N$43: now also R2.2; no longer R1.2
- net N$44: now also R3.2; no longer R2.2
- net N$45: now also R12.2; no longer R15.2
- net N$47: now also R30.2, R31.2; no longer R35.2, R36.2
- net N$48: now also R34.2; no longer R39.2
- net N$51: now also R35.2, R36.2; no longer R40.2, R41.2
- net N$52: now also R37.2, R38.2; no longer R42.2, R43.2
- net N$53: now also R32.2, R33.2; no longer R37.2, R38.2
- net N$54: now also R37.1; no longer R42.1
- net N$55: now also R18.1; no longer R23.1
- net N$57: now also C9.2; no longer C10.2
- net N$58: now also IC8.CK, R12.1; no longer BAT1.+, C29.2, IC8.VBAT
- net N$59: now also R20.2, R21.2; no longer R26.2, R27.2
- net N$6: now also R6.2, R7.1; no longer R10.1, R9.2
- net N$61: now also R31.1; no longer R36.1
- net N$62: now also R34.1; no longer R39.1
- net N$63: now also R33.1; no longer R38.1
- net N$65: now also C11.2; no longer C12.2
- net N$66: now also C11.1; no longer C12.1
- net N$68: now also C22.2, R20.1; no longer C221.2, R26.1
- net N$69: now also C22.1, R22.1; no longer C221.1, R28.1
- net N$7: now also R8.2, R9.1; no longer R11.2, R12.1
- net N$70: now also IC8.DI, R13.1; no longer IC8.!INT, R15.1, R18.2
- net N$71: now also R23.2; no longer R29.2
- net N$72: now also C10.1, R4.2, R5.2; no longer C11.1, R7.2, R8.2
- net N$73: now also R29.2; no longer IC8.SCL, R20.2
- net N$77: now also C20.2; no longer C22.2
- net N$79: now also R28.2; no longer IC8.SDA, R19.2
- net N$8: now also R45.2; no longer R6.2
- net N$80: now also R36.1; no longer R41.1
- net N$85: now also R16.1; no longer R21.1
- net N$9: now also R13.2; no longer R16.2
- net UVCC: now also C8.2; no longer C9.2
- net VCC: now also C10.2, C12.2, C29.1, C30.1, IC8.!HOLD, IC8.!WP, R1.1, R15.1, R17.1, R23.1, R27.1, R28.1, R38.1, R4.1, R43.2, R47.1; no longer C11.2, C15.2, C30.2, C33.2, R18.1, R20.1, R22.1, R24.1, R25.1, R3.1, R34.1, R35.1, R4.2, R43.1, R7.1
Other:
- moved on the sheet: C10, C11, C12, C13, C14, C15, C16, C17, C18, C19, C20, C21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
