File: rtu/eagle/rtu.brd (EAGLE design)
At the start: 76.2 x 65.4 mm, 114 parts

Commit message: do
Parts:
- removed D6: (no value), myparts:SOD123-DIODE
- D4: device myparts:SOT23-3 -> myparts:SOD123-DIODE
- IC7: device myparts:VSON-8 -> myparts:SOIC-8
- IC8: device myparts:WSON-8-6X5 -> myparts:SOIC-8-208
- moved D4 18.1 mm to (53.3, 32.0)
- moved D5 10.5 mm to (63.9, 32.0)
- moved R35 4.83 mm to (47.4, 15.9)
- moved R36 4.83 mm to (45.7, 15.9)
- moved R37 4.83 mm to (43.7, 15.9)
- moved R38 4.83 mm to (42.0, 15.9)
- moved IC7 2.65 mm to (43.9, 22.4)
- moved R46 0.40 mm to (14.9, 42.9)
- moved R47 0.40 mm to (14.9, 41.4)
- moved IC8 0.38 mm to (14.9, 37.5)
- moved C26 0.25 mm to (48.5, 23.7)
- moved C27 0.25 mm to (48.5, 25.3)
Connections:
- removed net N$53 (its old number): D4.2, F2.2, R36.1
- new net N$80: F2.2, R36.1
- net GND: no longer D4.3, IC7.9, IC8.9
- net N$28: now also D5.2; no longer D6.2
- net N$37: now also D4.2; no longer D5.2
- net N$54: no longer D4.1
- net VCC: now also D4.1; no longer D6.1
Routing:
- net N$53 (its old number): track 7.06 -> 0.00 mm
- net N$87: track 16.7 -> 10.5 mm, vias 2 -> 0
- net N$54: track 7.06 -> 1.76 mm
- net N$53: track 5.14 -> 7.73 mm
- net GND: track 78.8 -> 76.6 mm, vias 67 -> 64
- net N$80: track 0.00 -> 1.76 mm
- net N$25: track 7.72 -> 6.13 mm
- net N$51: track 3.77 -> 5.10 mm
- net N$47: track 3.40 -> 4.73 mm
- net N$52: track 3.77 -> 4.78 mm
- net VCC: track 270.8 -> 271.4 mm, vias 33 -> 31
- net N$57: vias 0 -> 2

Commit message: do
Parts:
- added BAT1: (no value), myparts:BAT-1220-BC501SM
- added C33: (no value), myparts:0603
- C10, C14, R27, R32: device myparts:0603 -> myparts:1206
- C12, C9, R25: device myparts:1206 -> myparts:0603
- C31: device myparts:CAPACITOR-SMD-8 -> myparts:0603
- C32: device myparts:0603 -> myparts:CAPACITOR-SMD-8
- IC3: device myparts:OPTO-SMD -> myparts:SOIC-8
- IC5: device myparts:VSSOP-10 -> myparts:OPTO-SMD
- IC7: device myparts:SOIC-8 -> myparts:VSSOP-10
- IC8: device myparts:SOIC-8-208 -> myparts:SOIC-8
- R16, R18, R36, R37: device myparts:0805 -> myparts:0603
- R21: device myparts:1206 -> myparts:0805
- R23, R41, R42: device myparts:0603 -> myparts:0805
- moved R46 57.5 mm to (71.2, 31.6), turned to 90 degrees
- moved R47 55.7 mm to (69.7, 31.6), turned to 270 degrees
- moved R30 54.3 mm to (3.94, -5.21), turned to 0 degrees
- moved C19 54.3 mm to (3.94, -30.7), turned to 0 degrees
- moved R7 52.7 mm to (11.8, 16.3), turned to 270 degrees
- moved C20 52.5 mm to (3.94, -33.0)
- moved R8 52.0 mm to (10.3, 13.3), turned to 90 degrees
- moved C21 49.8 mm to (3.94, -28.4)
- moved R18 48.1 mm to (3.94, -35.3), turned to 0 degrees
- moved C15 42.1 mm to (6.35, 32.5)
- moved IC3 41.9 mm to (3.68, -24.3), turned to 0 degrees
- moved R44 41.9 mm to (60.7, 31.6), turned to 90 degrees
- moved C18 40.2 mm to (54.0, 36.4)
- moved R45 39.9 mm to (59.2, 31.6), turned to 270 degrees
- moved R6 39.3 mm to (21.3, 44.3), turned to 180 degrees
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Connections:
- removed net N$64: CON5.5, R21.1, R22.2
- removed net N$86: IC1.41, R46.1
- removed net N$87: IC8.2, R14.1
- new net N$23: IC6.3, R16.1, R25.2
- new net N$81: CON5.5, R27.1, R28.2
- net GND: now also BAT1.-, C10.1, C22.1, C25.1, C28.1, C30.1, C33.1, C8.2, IC3.5, IC5.3, IC6.2, IC7.1, IC7.7, IC8.5, R37.1, R47.1, R6.1, R8.1; no longer C12.1, C26.1, C28.2, C29.2, C30.2, C8.1, IC3.3, IC5.1, IC5.2, IC5.7, IC7.5, IC8.4, R32.1, R35.1, R42.1, R5.1
- net N$1: now also IC1.41, R5.1; no longer IC1.40, R44.1
- net N$13: now also C17.2, R10.2, R12.2, R14.2; no longer C15.2, R11.2, R7.2, R9.2
- net N$14: now also R9.1; no longer R6.1
- net N$15: now also R5.2; no longer R44.2
- net N$16: now also R11.1; no longer R8.1
- net N$17: now also C29.1, IC7.8, IC7.9, R33.2; no longer C25.1, IC6.8, IC6.9, R26.2
- net N$18: now also R1.1; no longer R2.1
- net N$19: now also R2.1; no longer R3.1
- net N$2: now also C18.2, R13.1, R14.1; no longer C17.2, R10.1, R11.1
- net N$20: now also IC4.1, R21.2; no longer IC3.1, R16.2
- net N$21: now also C29.2, IC7.10, R31.2; no longer C25.2, IC6.10, R24.2
- net N$22: now also R13.2; no longer R10.2
- net N$24: now also R46.2; no longer R41.2
- net N$25: now also IC7.3, R17.1, R30.2; no longer IC8.1, R46.2, R47.2
- net N$26: now also R46.1, R47.2; no longer R41.1, R42.2
- net N$27: now also R34.2; no longer R27.2
- net N$29: now also C8.1, R4.1; no longer C28.1, R43.1
- net N$3: now also R17.2; no longer R14.2, R15.2
- net N$30: now also R31.1, R32.1; no longer R24.1, R25.1
- net N$32: now also C23.2, IC5.4, R24.2; no longer C19.2, IC4.4, R19.2
- net N$33: now also IC5.1, R23.2; no longer IC4.1, R18.2
- net N$35: now also C22.2, IC4.4, R22.2; no longer C18.2, IC3.4, R17.2
- net N$36: now also R44.1, R45.2; no longer R39.1, R40.2
- net N$38: now also R44.2; no longer R39.2
- net N$40: now also R32.2, R33.1; no longer R25.2, R26.1
- net N$41: now also R3.2; no longer R1.2
- net N$42: now also C27.2, C28.2, IC7.6; no longer C23.2, C24.2, IC6.6
- net N$43: now also R1.2; no longer R2.2
- net N$44: now also R2.2; no longer R3.2
- net N$45: now also R15.2; no longer R12.2
- net N$47: now also IC8.1, R35.2, R36.2; no longer IC7.1, R30.2, R31.2
- net N$48: now also IC8.4, R39.2; no longer IC7.4, R34.2
- net N$49: now also IC5.2; no longer IC4.2
- net N$50: now also IC4.2; no longer IC3.2
- net N$51: now also IC8.7, R40.2, R41.2; no longer IC7.7, R35.2, R36.2
- net N$52: now also IC8.6, R42.2, R43.2; no longer IC7.6, R37.2, R38.2
- net N$53: now also IC8.2, IC8.3, R37.2, R38.2; no longer IC7.2, IC7.3, R32.2, R33.2
- net N$54: now also R42.1; no longer R37.1
- net N$55: now also R23.1; no longer R18.1
- net N$57: now also C10.2; no longer C9.2
- net N$58: now also BAT1.+, C21.2, IC3.6; no longer IC8.6, R12.1
- net N$59: now also R26.2, R27.2; no longer R20.2, R21.2
- net N$6: now also R10.1, R9.2; no longer R6.2, R7.1
- net N$61: now also R36.1; no longer R31.1
- net N$62: now also R39.1; no longer R34.1
- net N$63: now also R38.1; no longer R33.1
- net N$65: now also C12.2; no longer C11.2
- net N$66: now also C12.1; no longer C11.1
- net N$68: now also C26.2, IC6.10, R26.1; no longer C22.2, IC5.10, R20.1
- net N$69: now also C26.1, IC6.8, IC6.9, R28.1; no longer C22.1, IC5.8, IC5.9, R22.1
- net N$7: now also R11.2, R12.1; no longer R8.2, R9.1
- net N$70: now also IC3.3, R15.1, R18.2; no longer IC8.5, R13.1
- net N$71: now also R29.2; no longer R23.2
- net N$72: now also C11.1, R7.2, R8.2; no longer C10.1, R4.2, R5.2
- net N$73: now also IC3.8, IC7.5, R20.2; no longer IC5.5, R29.2
- net N$77: now also C24.2, C25.2, IC6.6; no longer C20.2, C21.2, IC5.6
- net N$79: now also IC3.7, IC7.4, R19.2; no longer IC5.4, R28.2
- net N$8: now also R6.2; no longer R45.2
- net N$80: now also R41.1; no longer R36.1
- net N$85: now also R21.1; no longer R16.1
- net N$9: now also R16.2; no longer R13.2
- net UVCC: now also C9.2; no longer C8.2
- net VCC: now also C11.2, C15.2, C19.2, C20.2, C30.2, C33.2, IC3.2, IC7.2, R18.1, R20.1, R22.1, R24.1, R25.1, R3.1, R34.1, R35.1, R4.2, R43.1, R7.1; no longer C10.2, C12.2, C26.2, C27.2, C29.1, C30.1, IC6.2, IC7.8, IC8.3, IC8.7, R1.1, R15.1, R17.1, R23.1, R27.1, R28.1, R38.1, R4.1, R43.2, R47.1
Routing:
- net VCC: track 271.4 -> 241.7 mm, vias 31 -> 28
- net N$86: track 22.2 -> 0.00 mm, vias 2 -> 0
- net N$87: track 10.5 -> 0.00 mm
- net N$3: track 16.1 -> 6.81 mm, vias 1 -> 0
- net N$9: track 18.3 -> 11.8 mm
- net N$25: track 6.13 -> 0.00 mm
- net GND: track 76.6 -> 72.5 mm, vias 64 -> 62
- net N$64: track 3.68 -> 0.00 mm
- net N$45: track 13.5 -> 10.1 mm
- net N$70: track 2.32 -> 0.00 mm
- net N$58: track 2.21 -> 0.00 mm
- net N$81: track 0.00 -> 2.15 mm

Commit message: do
Parts:
- moved BAT1 92.9 mm to (16.9, 48.6), turned to 270 degrees
- moved R18 75.6 mm to (21.3, 38.2), turned to 180 degrees
- moved C20 71.7 mm to (14.0, 38.0)
- moved C19 69.8 mm to (13.0, 38.5)
- moved IC3 58.6 mm to (14.2, 33.4), turned to 270 degrees
- moved C21 57.6 mm to (14.2, 28.2)
- moved R30 37.1 mm to (23.9, 26.0)
- moved R25 33.1 mm to (19.9, 26.0)
- moved R17 9.03 mm to (23.9, 27.6), turned to 180 degrees
- moved R16 6.31 mm to (19.9, 27.6), turned to 180 degrees
- moved R5 4.91 mm to (26.2, 45.0)
- moved R6 4.91 mm to (26.2, 43.4)
Routing:
- net N$25: track 0.00 -> 21.9 mm, vias 0 -> 2
- net N$23: track 0.00 -> 17.5 mm, vias 0 -> 2
- net N$1: track 17.6 -> 11.1 mm, vias 2 -> 0
- net N$3: track 6.81 -> 12.2 mm
- net N$15: track 22.0 -> 27.1 mm, vias 0 -> 2
- net N$8: track 27.8 -> 32.4 mm, vias 0 -> 2
- net N$9: track 11.8 -> 15.8 mm
- net N$45: track 10.1 -> 13.9 mm
- net GND: track 72.5 -> 74.3 mm, vias 62 -> 60
- net VCC: track 241.7 -> 240.2 mm, vias 28 -> 26
- net N$41: track 55.7 -> 54.9 mm, vias 2 -> 3
- net N$56: track 40.9 -> 40.0 mm
- net N$19: track 27.3 -> 26.7 mm
- net N$18: track 25.5 -> 24.9 mm

Commit message: do
Parts:
- moved R15 2.07 mm to (19.9, 35.2)
- moved R18 2.07 mm to (19.9, 36.7)
- moved C21 1.40 mm to (14.1, 26.8), turned to 90 degrees
- moved C20 0.99 mm to (13.3, 37.2)
- moved IC3 0.89 mm to (14.2, 32.5)
- moved C19 0.46 mm to (13.3, 38.7)
Routing:
- net VCC: track 240.2 -> 262.6 mm, vias 26 -> 28
- net N$79: track 29.6 -> 51.1 mm, vias 0 -> 4
- net N$73: track 32.3 -> 53.5 mm, vias 4 -> 8
- net N$58: track 0.00 -> 16.5 mm
- net N$70: track 0.00 -> 13.9 mm, vias 0 -> 2
- net GND: track 74.3 -> 82.5 mm, vias 60 -> 64
- net N$23: track 17.5 -> 18.6 mm
- net N$45: track 13.9 -> 14.9 mm
- net N$25: track 21.9 -> 22.7 mm
- added copper zone on layer 1, net N$81
- removed copper zone on layer 1, net N$64

Commit message: do
Parts:
- moved C22 0.51 mm to (16.5, 20.6)
- moved IC4 0.51 mm to (16.5, 15.5)
- moved R21 0.51 mm to (16.5, 9.53)
- moved R22 0.51 mm to (16.5, 22.1)
Routing:
- net GND: track 82.5 -> 96.6 mm, vias 64 -> 67
- net N$81: track 2.15 -> 3.68 mm
- net VCC: track 262.6 -> 261.2 mm
- net N$35: track 42.4 -> 42.9 mm

Commit message: do
Routing:
- net VCC: track 261.2 -> 259.8 mm

Commit message: do
Parts:
- removed D4, D5: (no value), myparts:SOD123-DIODE
- removed Q1, Q2: (no value), myparts:SOT23-3
- removed R44, R45, R46, R47: (no value), myparts:0603
- added IC10, IC9: (no value), myparts:SC74-6
- SW3, SW4: device myparts:HK19F -> myparts:HFD2-L2
- moved C33 1.14 mm to (36.7, 43.2)
Connections:
- removed net N$36: Q1.1, R44.1, R45.2
- removed net N$37: D4.2, Q1.3, SW3.L2
- new net N$64: IC10.6, SW4.L1-
- new net N$82: IC10.3, SW4.L2-
- new net N$90: IC1.38, IC9.5
- new net N$91: IC1.39, IC9.2
- net GND: now also IC10.1, IC10.4, IC9.1, IC9.4; no longer Q1.2, Q2.2, R45.1, R47.1
- net N$24: now also IC1.36, IC10.5; no longer IC1.27, R46.2
- net N$26: now also IC9.6, SW3.L1-; no longer Q2.1, R46.1, R47.2
- net N$28: now also IC9.3, SW3.L2-; no longer D5.2, Q2.3, SW4.L2
- net N$32: now also IC1.28; no longer IC1.29
- net N$35: now also IC1.29; no longer IC1.28
- net N$38: now also IC1.37, IC10.2; no longer IC1.26, R44.2
- net VCC: now also SW3.L1+, SW3.L2+, SW4.L1+, SW4.L2+; no longer D4.1, D5.1, SW3.L1, SW4.L1
Routing:
- net N$90: track 0.00 -> 32.1 mm, vias 0 -> 2
- net N$91: track 0.00 -> 27.3 mm, vias 0 -> 2
- net N$38: track 25.1 -> 38.2 mm, vias 0 -> 2
- net N$37: track 10.9 -> 0.00 mm
- net N$82: track 0.00 -> 8.92 mm
- net N$64: track 0.00 -> 7.22 mm
- net N$32: track 40.1 -> 34.7 mm
- net N$26: track 3.13 -> 7.22 mm
- net N$14: track 27.1 -> 23.9 mm
- net N$36: track 3.13 -> 0.00 mm
- net N$61: track 18.2 -> 15.2 mm
- net N$24: track 36.7 -> 39.6 mm, vias 0 -> 2
- net N$16: track 22.6 -> 19.8 mm
- net N$28: track 11.3 -> 8.84 mm
- net GND: track 96.3 -> 98.0 mm, vias 67 -> 69
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
Commit message: do
Routing:
- net GND: vias 69 -> 70
Changed lines of the file:
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@@
 <contactref element="SW2" pad="4"/>
 <contactref element="SW2" pad="3"/>
-<via x="19.685" y="59.563" extent="1-16" drill="0.4"/>
+<via x="19.685" y="59.563" extent="1-16" drill="0.6"/>
 <wire x1="24.384" y1="39.751" x2="25.4" y2="39.751" width="0.3048" layer="1"/>
 <contactref element="SW2" pad="2"/>
@@
 <wire x1="68.326" y1="30.546" x2="69.657" y2="30.546" width="0.508" layer="1"/>
 <wire x1="69.657" y1="30.546" x2="69.723" y2="30.48" width="0.508" layer="1"/>
+<via x="42.164" y="58.039" extent="1-16" drill="1.1"/>
 </signal>
 <signal name="N$2">
@@
 <wire x1="10.033" y1="19.431" x2="10.033" y2="24.638" width="1.016" layer="16"/>
 <via x="6.604" y="42.799" extent="1-16" drill="0.7"/>
-<wire x1="6.604" y1="42.799" x2="6.604" y2="47.244" width="2.032" layer="1"/>
+<wire x1="6.604" y1="42.799" x2="6.604" y2="46.863" width="2.032" layer="1"/>
 <via x="8.509" y="32.512" extent="1-16" drill="0.7"/>
 <wire x1="8.509" y1="34.036" x2="8.509" y2="32.512" width="2.032" layer="16"/>
@@
 <wire x1="26.416" y1="49.149" x2="28.194" y2="49.149" width="2.032" layer="1"/>
 <wire x1="31.242" y1="46.736" x2="34.544" y2="46.736" width="2.032" layer="1"/>
-<wire x1="6.604" y1="47.244" x2="8.636" y2="49.276" width="2.032" layer="1"/>
-<wire x1="8.636" y1="49.276" x2="11.43" y2="49.276" width="2.032" layer="1"/>
+<wire x1="6.604" y1="46.863" x2="8.89" y2="49.149" width="2.032" layer="1"/>
+<wire x1="8.89" y1="49.149" x2="11.43" y2="49.149" width="2.032" layer="1"/>
 <wire x1="11.43" y1="49.149" x2="20.574" y2="49.149" width="2.032" layer="1"/>
 <wire x1="26.416" y1="49.149" x2="20.574" y2="49.149" width="2.032" layer="16"/>
@@
 <wire x1="23.114" y1="26.035" x2="23.114" y2="24.892" width="0.3048" layer="1"/>
 <wire x1="23.114" y1="24.892" x2="23.368" y2="24.638" width="0.3048" layer="1"/>
-<wire x1="11.43" y1="53.975" x2="11.43" y2="49.276" width="0.508" layer="1"/>
-<wire x1="11.43" y1="49.276" x2="11.43" y2="49.149" width="0.508" layer="1"/>
+<wire x1="11.43" y1="53.975" x2="11.43" y2="49.149" width="0.508" layer="1"/>
 <wire x1="14.097" y1="38.735" x2="14.097" y2="37.211" width="0.762" layer="1"/>
 <wire x1="24.892" y1="29.337" x2="24.384" y2="29.845" width="0.6096" layer="1"/>
@@
 <wire x1="52.324" y1="27.686" x2="52.324" y2="25.146" width="1.016" layer="1"/>
 <wire x1="63.246" y1="27.686" x2="63.246" y2="25.146" width="1.016" layer="1"/>
-<wire x1="52.324" y1="25.146" x2="55.626" y2="25.146" width="1.016" layer="1"/>
-<wire x1="55.626" y1="25.146" x2="57.531" y2="23.241" width="1.016" layer="1"/>
-<wire x1="57.531" y1="23.241" x2="61.341" y2="23.241" width="1.016" layer="1"/>
+<wire x1="52.324" y1="25.146" x2="55.118" y2="25.146" width="1.016" layer="1"/>
+<wire x1="55.118" y1="25.146" x2="57.023" y2="23.241" width="1.016" layer="1"/>
+<wire x1="57.023" y1="23.241" x2="61.341" y2="23.241" width="1.016" layer="1"/>
 <wire x1="61.341" y1="23.241" x2="63.246" y2="25.146" width="1.016" layer="1"/>
 <wire x1="47.752" y1="26.67" x2="48.768" y2="26.67" width="1.016" layer="1"/>
@@
 <wire x1="5.715" y1="41.021" x2="4.826" y2="41.021" width="0.508" layer="1"/>
 <wire x1="4.826" y1="41.021" x2="4.826" y2="39.116" width="0.8128" layer="1"/>
-<wire x1="21.336" y1="46.228" x2="10.033" y2="46.228" width="0.8128" layer="1"/>
-<wire x1="9.652" y1="45.847" x2="9.652" y2="45.085" width="0.8128" layer="1"/>
-<wire x1="10.033" y1="46.228" x2="9.652" y2="45.847" width="0.8128" layer="1"/>
+<wire x1="21.336" y1="46.228" x2="10.287" y2="46.228" width="0.8128" layer="1"/>
+<wire x1="9.652" y1="45.593" x2="9.652" y2="45.085" width="0.8128" layer="1"/>
+<wire x1="10.287" y1="46.228" x2="9.652" y2="45.593" width="0.8128" layer="1"/>
 </signal>
 <signal name="N$34">
@@
 <wire x1="9.3694" y1="41.7366" x2="8.4582" y2="42.6478" width="1.016" layer="1"/>
 <wire x1="9.3694" y1="39.5954" x2="8.89" y2="39.116" width="1.016" layer="1"/>
-<wire x1="8.4582" y1="46.4312" x2="9.398" y2="47.371" width="1.016" layer="1"/>
-<wire x1="9.398" y1="47.371" x2="21.209" y2="47.371" width="1.016" layer="1"/>
-<wire x1="8.4582" y1="42.6478" x2="8.4582" y2="46.4312" width="1.016" layer="1"/>
+<wire x1="8.4582" y1="46.0502" x2="9.779" y2="47.371" width="1.016" layer="1"/>
+<wire x1="9.779" y1="47.371" x2="21.209" y2="47.371" width="1.016" layer="1"/>
+<wire x1="8.4582" y1="42.6478" x2="8.4582" y2="46.0502" width="1.016" layer="1"/>
 <wire x1="24.511" y1="47.371" x2="24.511" y2="56.642" width="1.016" layer="1"/>
 <wire x1="23.241" y1="57.912" x2="24.511" y2="56.642" width="1.016" layer="1"/>
@@
 <contactref element="R16" pad="1"/>
 <via x="28.956" y="17.526" extent="1-16" drill="0.4"/>
-<wire x1="29.591" y1="19.2405" x2="29.591" y2="18.034" width="0.3048" layer="1"/>
-<wire x1="29.591" y1="18.034" x2="29.083" y2="17.526" width="0.3048" layer="1"/>
-<wire x1="29.083" y1="17.526" x2="28.956" y2="17.526" width="0.3048" layer="1"/>
+<wire x1="29.591" y1="19.2405" x2="29.591" y2="18.161" width="0.3048" layer="1"/>
+<wire x1="29.591" y1="18.161" x2="28.956" y2="17.526" width="0.3048" layer="1"/>
 <via x="21.717" y="25.781" extent="1-16" drill="0.4"/>
 <wire x1="28.956" y1="17.526" x2="28.194" y2="18.288" width="0.3048" layer="16"/>
@@
 <contactref element="R17" pad="1"/>
 <via x="37.084" y="17.526" extent="1-16" drill="0.4"/>
-<wire x1="37.719" y1="19.2405" x2="37.719" y2="18.034" width="0.3048" layer="1"/>
-<wire x1="37.211" y1="17.526" x2="37.084" y2="17.526" width="0.3048" layer="1"/>
-<wire x1="37.719" y1="18.034" x2="37.211" y2="17.526" width="0.3048" layer="1"/>
+<wire x1="37.719" y1="19.2405" x2="37.719" y2="18.161" width="0.3048" layer="1"/>
+<wire x1="37.719" y1="18.161" x2="37.084" y2="17.526" width="0.3048" layer="1"/>
 <via x="25.654" y="25.781" extent="1-16" drill="0.4"/>
 <wire x1="37.084" y1="17.526" x2="34.163" y2="17.526" width="0.3048" layer="16"/>
@@
 <wire x1="46.274775" y1="34.1598" x2="49.2792" y2="34.1598" width="0.3048" layer="16"/>
 <wire x1="44.366575" y1="36.068" x2="46.274775" y2="34.1598" width="0.3048" layer="16"/>
-<wire x1="49.53" y1="33.909" x2="49.7872" y2="33.6518" width="0.3048" layer="1"/>
-<wire x1="49.7872" y1="33.6518" x2="49.84430625" y2="33.6518" width="0.3048" layer="1"/>
-<wire x1="49.84430625" y1="33.6518" x2="49.97130625" y2="33.5248" width="0.3048" layer="1"/>
+<wire x1="49.97130625" y1="33.5248" x2="49.58710625" y2="33.909" width="0.3048" layer="1"/>
+<wire x1="49.53" y1="33.909" x2="49.58710625" y2="33.909" width="0.3048" layer="1"/>
 <wire x1="52.491375" y1="33.5248" x2="53.002575" y2="34.036" width="0.3048" layer="1"/>
 <wire x1="49.97130625" y1="33.5248" x2="52.491375" y2="33.5248" width="0.3048" layer="1"/>
