File: rtu/eagle/rtu.brd (EAGLE design)
At the start: 76.2 x 65.4 mm, 109 parts

Commit message: do
Parts:
- moved C5 0.81 mm to (30.6, 42.5)
Connections:
- new net N$36: IC1.41, R6.1
- net GND: no longer R6.1
- net N$1: now also IC1.40; no longer IC1.41
Routing:
- net N$36: track 0.00 -> 10.2 mm
- net N$91: track 27.3 -> 31.4 mm
- net N$90: track 32.1 -> 33.0 mm
- net N$31: track 3.62 -> 4.27 mm
- net GND: vias 70 -> 68
Changed lines of the file:
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@@
 <attribute name="VALUE" x="38.989" y="23.749" size="1.016" layer="27" rot="R180"/>
 </element>
-<element name="C5" library="myparts" package="0603" value="" x="31.242" y="42.037" smashed="yes">
-<attribute name="NAME" x="31.242" y="43.18" size="0.8128" layer="25" align="center"/>
-<attribute name="VALUE" x="27.813" y="41.783" size="1.016" layer="27"/>
+<element name="C5" library="myparts" package="0603" value="" x="30.607" y="42.545" smashed="yes">
+<attribute name="NAME" x="30.607" y="43.688" size="0.8128" layer="25" align="center"/>
+<attribute name="VALUE" x="27.178" y="42.291" size="1.016" layer="27"/>
 </element>
 <element name="C6" library="myparts" package="0603" value="" x="26.162" y="35.179" smashed="yes">
@@
 <contactref element="D3" pad="2"/>
 <contactref element="C8" pad="2"/>
-<contactref element="R6" pad="1"/>
 <contactref element="IC1" pad="33"/>
 <contactref element="C31" pad="1"/>
@@
 <wire x1="32.29" y1="40.481" x2="32.004" y2="40.767" width="0.3048" layer="1"/>
 <via x="24.384" y="39.751" extent="1-16" drill="0.4"/>
-<via x="32.004" y="43.307" extent="1-16" drill="0.4"/>
-<wire x1="32.004" y1="43.307" x2="30.734" y2="43.307" width="0.3048" layer="1"/>
-<wire x1="30.734" y1="43.307" x2="30.48" y2="43.053" width="0.3048" layer="1"/>
-<wire x1="30.48" y1="43.053" x2="30.48" y2="42.037" width="0.3048" layer="1"/>
 <via x="46.355" y="36.449" extent="1-16" drill="0.4"/>
 <contactref element="SW1" pad="2"/>
@@
 <wire x1="50.292" y1="25.273" x2="49.276" y2="25.273" width="0.508" layer="1"/>
 <contactref element="C33" pad="1"/>
-<via x="34.925" y="43.18" extent="1-16" drill="0.4"/>
+<via x="34.925" y="43.688" extent="1-16" drill="0.4"/>
 <via x="48.387" y="15.113" extent="1-16" drill="0.4"/>
 <wire x1="48.387" y1="15.113" x2="47.371" y2="15.113" width="0.3048" layer="1"/>
@@
 <wire x1="22.352" y1="20.066" x2="22.86" y2="19.558" width="0.3048" layer="1"/>
 <wire x1="23.368" y1="20.574" x2="22.352" y2="20.574" width="0.3048" layer="1"/>
-<wire x1="35.941" y1="43.18" x2="34.925" y2="43.18" width="0.3048" layer="1"/>
+<wire x1="35.941" y1="43.18" x2="35.306" y2="43.18" width="0.3048" layer="1"/>
+<wire x1="35.306" y1="43.18" x2="34.925" y2="43.561" width="0.3048" layer="1"/>
+<wire x1="34.925" y1="43.561" x2="34.925" y2="43.688" width="0.3048" layer="1"/>
 <polygon width="0" layer="1" thermals="no">
 <vertex x="9.779" y="13.081"/>
@@
 </polygon>
 <via x="10.287" y="11.557" extent="1-16" drill="0.4"/>
-<via x="27.94" y="43.434" extent="1-16" drill="0.4"/>
-<wire x1="26.924" y1="43.434" x2="27.94" y2="43.434" width="0.3048" layer="1"/>
 <contactref element="CON5" pad="11"/>
 <contactref element="IC8" pad="5"/>
@@
 <wire x1="69.657" y1="30.546" x2="69.723" y2="30.48" width="0.508" layer="1"/>
 <via x="42.164" y="58.039" extent="1-16" drill="1.1"/>
+<wire x1="30.1022" y1="41.5258" x2="29.845" y2="41.783" width="0.3048" layer="1"/>
+<wire x1="29.845" y1="42.545" x2="29.845" y2="41.783" width="0.3048" layer="1"/>
+<wire x1="31.2452" y1="41.5258" x2="32.004" y2="40.767" width="0.3048" layer="1"/>
+<wire x1="30.1022" y1="41.5258" x2="31.2452" y2="41.5258" width="0.3048" layer="1"/>
 </signal>
 <signal name="N$2">
@@
 <contactref element="IC1" pad="42"/>
 <contactref element="C5" pad="2"/>
-<wire x1="32.79" y1="41.886" x2="32.639" y2="42.037" width="0.3048" layer="1"/>
-<wire x1="32.639" y1="42.037" x2="32.004" y2="42.037" width="0.3048" layer="1"/>
-<wire x1="32.79" y1="41.886" x2="32.79" y2="39.116" width="0.3048" layer="1"/>
+<wire x1="32.79" y1="41.124" x2="32.258" y2="41.656" width="0.3048" layer="1"/>
+<wire x1="32.258" y1="41.656" x2="31.833425" y2="41.656" width="0.3048" layer="1"/>
+<wire x1="31.369" y1="42.120425" x2="31.369" y2="42.545" width="0.3048" layer="1"/>
+<wire x1="32.79" y1="39.116" x2="32.79" y2="41.124" width="0.3048" layer="1"/>
+<wire x1="31.833425" y1="41.656" x2="31.369" y2="42.120425" width="0.3048" layer="1"/>
 </signal>
 <signal name="UVCC">
@@
 <signal name="N$1">
 <contactref element="R5" pad="1"/>
-<contactref element="IC1" pad="41"/>
-<wire x1="32.31830625" y1="44.0658" x2="32.0072" y2="44.0658" width="0.3048" layer="1"/>
-<wire x1="32.0072" y1="44.0658" x2="32.004" y2="44.069" width="0.3048" layer="1"/>
-<wire x1="33.29" y1="43.09410625" x2="32.31830625" y2="44.0658" width="0.3048" layer="1"/>
-<wire x1="32.004" y1="44.069" x2="28.448" y2="44.069" width="0.3048" layer="1"/>
-<wire x1="27.559" y1="44.958" x2="26.924" y2="44.958" width="0.3048" layer="1"/>
-<wire x1="33.29" y1="39.116" x2="33.29" y2="43.09410625" width="0.3048" layer="1"/>
-<wire x1="28.448" y1="44.069" x2="27.559" y2="44.958" width="0.3048" layer="1"/>
+<wire x1="26.924" y1="44.958" x2="27.559" y2="44.958" width="0.3048" layer="1"/>
+<contactref element="IC1" pad="40"/>
+<wire x1="28.448" y1="44.069" x2="32.341425" y2="44.069" width="0.3048" layer="1"/>
+<wire x1="27.559" y1="44.958" x2="28.448" y2="44.069" width="0.3048" layer="1"/>
+<wire x1="32.341425" y1="44.069" x2="32.893" y2="43.517425" width="0.3048" layer="1"/>
+<wire x1="32.893" y1="42.501425" x2="32.893" y2="43.517425" width="0.3048" layer="1"/>
+<wire x1="33.79" y1="39.116" x2="33.79" y2="41.604425" width="0.3048" layer="1"/>
+<wire x1="33.79" y1="41.604425" x2="32.893" y2="42.501425" width="0.3048" layer="1"/>
 </signal>
 <signal name="N$17" airwireshidden="yes">
@@
 <signal name="N$90">
 <contactref element="IC1" pad="38"/>
-<via x="34.671" y="42.164" extent="1-16" drill="0.4"/>
+<via x="34.671" y="42.672" extent="1-16" drill="0.4"/>
 <wire x1="34.79" y1="39.116" x2="34.79" y2="40.759" width="0.3048" layer="1"/>
-<wire x1="35.052" y1="41.45910625" x2="34.671" y2="41.84010625" width="0.3048" layer="1"/>
-<wire x1="34.671" y1="41.84010625" x2="34.671" y2="42.164" width="0.3048" layer="1"/>
-<wire x1="35.052" y1="41.021" x2="35.052" y2="41.45910625" width="0.3048" layer="1"/>
-<wire x1="34.79" y1="40.759" x2="35.052" y2="41.021" width="0.3048" layer="1"/>
-<wire x1="34.671" y1="42.164" x2="34.9282" y2="41.9068" width="0.3048" layer="16"/>
-<wire x1="34.9282" y1="41.9068" x2="34.9282" y2="41.25826875" width="0.3048" layer="16"/>
+<wire x1="34.925" y1="42.418" x2="34.671" y2="42.672" width="0.3048" layer="1"/>
+<wire x1="34.925" y1="42.418" x2="34.925" y2="40.894" width="0.3048" layer="1"/>
+<wire x1="34.79" y1="40.759" x2="34.925" y2="40.894" width="0.3048" layer="1"/>
+<wire x1="34.671" y1="42.672" x2="34.9282" y2="42.4148" width="0.3048" layer="16"/>
+<wire x1="34.9282" y1="42.4148" x2="34.9282" y2="41.25826875" width="0.3048" layer="16"/>
 <wire x1="36.05446875" y1="40.132" x2="36.35204375" y2="40.132" width="0.3048" layer="16"/>
 <wire x1="36.35204375" y1="40.132" x2="38.63484375" y2="37.8492" width="0.3048" layer="16"/>
@@
 <signal name="N$91">
 <contactref element="IC1" pad="39"/>
-<via x="34.163" y="41.275" extent="1-16" drill="0.4"/>
-<wire x1="34.29" y1="39.116" x2="34.29" y2="41.148" width="0.3048" layer="1"/>
-<wire x1="34.29" y1="41.148" x2="34.163" y2="41.275" width="0.3048" layer="1"/>
-<wire x1="34.163" y1="41.275" x2="35.8108" y2="39.6272" width="0.3048" layer="16"/>
-<wire x1="35.8108" y1="39.6272" x2="35.84084375" y2="39.6272" width="0.3048" layer="16"/>
-<wire x1="35.84084375" y1="39.6272" x2="35.84404375" y2="39.624" width="0.3048" layer="16"/>
-<wire x1="35.84404375" y1="39.624" x2="36.14161875" y2="39.624" width="0.3048" layer="16"/>
+<via x="33.782" y="43.18" extent="1-16" drill="0.4"/>
+<wire x1="36.14161875" y1="39.624" x2="35.84404375" y2="39.624" width="0.3048" layer="16"/>
 <wire x1="36.14161875" y1="39.624" x2="38.42441875" y2="37.3412" width="0.3048" layer="16"/>
 <wire x1="38.42441875" y1="37.3412" x2="39.624525" y2="37.3412" width="0.3048" layer="16"/>
@@
 <wire x1="53.213" y1="31.496" x2="52.2002" y2="32.5088" width="0.3048" layer="1"/>
 <wire x1="52.2002" y1="32.5088" x2="50.6698" y2="32.5088" width="0.3048" layer="1"/>
+<wire x1="33.782" y1="42.418" x2="33.782" y2="43.18" width="0.3048" layer="1"/>
+<wire x1="34.29" y1="39.116" x2="34.29" y2="41.91" width="0.3048" layer="1"/>
+<wire x1="34.29" y1="41.91" x2="33.782" y2="42.418" width="0.3048" layer="1"/>
+<wire x1="35.84404375" y1="39.624" x2="34.4202" y2="41.04784375" width="0.3048" layer="16"/>
+<wire x1="33.782" y1="42.418" x2="33.782" y2="43.18" width="0.3048" layer="16"/>
+<wire x1="34.4202" y1="41.04784375" x2="34.4202" y2="41.7798" width="0.3048" layer="16"/>
+<wire x1="34.4202" y1="41.7798" x2="33.782" y2="42.418" width="0.3048" layer="16"/>
+</signal>
+<signal name="N$36">
+<contactref element="R6" pad="1"/>
+<contactref element="IC1" pad="41"/>
+<wire x1="26.924" y1="43.434" x2="27.051" y2="43.561" width="0.3048" layer="1"/>
+<wire x1="27.051" y1="43.561" x2="32.131" y2="43.561" width="0.3048" layer="1"/>
+<wire x1="32.385" y1="43.307" x2="32.131" y2="43.561" width="0.3048" layer="1"/>
+<wire x1="33.29" y1="39.116" x2="33.29" y2="41.386" width="0.3048" layer="1"/>
+<wire x1="33.29" y1="41.386" x2="32.385" y2="42.291" width="0.3048" layer="1"/>
+<wire x1="32.385" y1="42.291" x2="32.385" y2="43.307" width="0.3048" layer="1"/>
 </signal>
 </signals>

Commit message: do
Connections:
- net N$36: now also IC1.12; no longer IC1.41
Routing:
- net N$36: track 10.2 -> 27.7 mm, vias 0 -> 4
