File: rtu/eagle/rtu.sch (EAGLE design)
At the start: 114 parts

Commit message: do
Parts:
- removed D6: (no value), myparts:DIODE-SCHOTTKY
- D4: device myparts:TVS-DIODE-3P -> myparts:DIODE-SCHOTTKY
- IC7: device myparts:SN65HVD72DRB -> myparts:IC-485-HALF
- IC8: device myparts:MEM-SPI-WSON-8-6X5 -> myparts:MEM-SPI-SOIC-8-208
Connections:
- removed net N$53 (its old number): D4.2, F2.2, R36.1
- new net N$80: F2.2, R36.1
- net GND: no longer D4.3, IC7.EP, IC8.EP
- net N$28: now also D5.A; no longer D6.A
- net N$37: now also D4.A; no longer D5.A
- net N$54: no longer D4.1
- net VCC: now also D4.K; no longer D6.K
Other:
- moved on the sheet: CON6, D5, F2, F3, Q1, Q2, R39, R40, R41, R42, SW3, SW4

Commit message: do
Parts:
- added BAT1: (no value), myparts:BAT-1220-BC501SM
- added C33: (no value), myparts:CAPACITOR-0603
- C10, C14: device myparts:CAPACITOR-0603 -> myparts:CAPACITOR-1206
- C12, C9: device myparts:CAPACITOR-1206 -> myparts:CAPACITOR-0603
- C31: device myparts:CAPACITOR-SMD-8 -> myparts:CAPACITOR-0603
- C32: device myparts:CAPACITOR-0603 -> myparts:CAPACITOR-SMD-8
- IC3: device myparts:OPTO-SMD -> myparts:DS3231M
- IC5: device myparts:INA226 -> myparts:OPTO-SMD
- IC7: device myparts:IC-485-HALF -> myparts:INA226
- IC8: device myparts:MEM-SPI-SOIC-8-208 -> myparts:IC-485-HALF
- R16, R18, R36, R37: device myparts:RESISTOR-0805 -> myparts:RESISTOR-0603
- R21: device myparts:RESISTOR-1206 -> myparts:RESISTOR-0805
- R23, R41, R42: device myparts:RESISTOR-0603 -> myparts:RESISTOR-0805
- R25: device myparts:RESISTOR-1206 -> myparts:RESISTOR-0603
- R27, R32: device myparts:RESISTOR-0603 -> myparts:RESISTOR-1206
Connections:
- removed net N$64: CON5.5, R21.1, R22.2
- removed net N$86: IC1.ADC0/PF0, R46.1
- removed net N$87: IC8.DO, R14.1
- new net N$23: IC6.ALR, R16.1, R25.2
- new net N$81: CON5.5, R27.1, R28.2
- net GND: now also BAT1.-, C10.1, C22.1, C25.1, C28.1, C30.1, C33.1, C8.2, IC3.GND, IC5.E, IC6.A0, IC7.A1, R37.1, R47.1, R6.1, R8.1; no longer C12.1, C26.1, C28.2, C29.2, C30.2, C8.1, IC3.E, IC5.A0, IC5.A1, IC5.GND, R32.1, R35.1, R42.1, R5.1
- net N$1: now also IC1.ADC0/PF0, R5.1; no longer IC1.ADC1/PF1, R44.1
- net N$13: now also C17.2, R10.2, R12.2, R14.2; no longer C15.2, R11.2, R7.2, R9.2
- net N$14: now also R9.1; no longer R6.1
- net N$15: now also R5.2; no longer R44.2
- net N$16: now also R11.1; no longer R8.1
- net N$17: now also C29.1, IC7.IN-, IC7.VBUS, R33.2; no longer C25.1, IC6.IN-, IC6.VBUS, R26.2
- net N$18: now also R1.1; no longer R2.1
- net N$19: now also R2.1; no longer R3.1
- net N$2: now also C18.2, R13.1, R14.1; no longer C17.2, R10.1, R11.1
- net N$20: now also IC4.A, R21.2; no longer IC3.A, R16.2
- net N$21: now also C29.2, IC7.IN+, R31.2; no longer C25.2, IC6.IN+, R24.2
- net N$22: now also R13.2; no longer R10.2
- net N$24: now also R46.2; no longer R41.2
- net N$25: now also IC7.ALR, R17.1, R30.2; no longer IC8.!CS, R46.2, R47.2
- net N$26: now also R46.1, R47.2; no longer R41.1, R42.2
- net N$27: now also R34.2; no longer R27.2
- net N$29: now also C8.1, R4.1; no longer C28.1, R43.1
- net N$3: now also R17.2; no longer R14.2, R15.2
- net N$30: now also R31.1, R32.1; no longer R24.1, R25.1
- net N$32: now also C23.2, IC5.C, R24.2; no longer C19.2, IC4.C, R19.2
- net N$33: now also IC5.A, R23.2; no longer IC4.A, R18.2
- net N$35: now also C22.2, IC4.C, R22.2; no longer C18.2, IC3.C, R17.2
- net N$36: now also R44.1, R45.2; no longer R39.1, R40.2
- net N$38: now also R44.2; no longer R39.2
- net N$40: now also R32.2, R33.1; no longer R25.2, R26.1
- net N$41: now also R3.2; no longer R1.2
- net N$42: now also C27.2, C28.2, IC7.VS; no longer C23.2, C24.2, IC6.VS
- net N$43: now also R1.2; no longer R2.2
- net N$44: now also R2.2; no longer R3.2
- net N$45: now also R15.2; no longer R12.2
- net N$47: now also IC8.R, R35.2, R36.2; no longer IC7.R, R30.2, R31.2
- net N$48: now also IC8.D, R39.2; no longer IC7.D, R34.2
- net N$49: now also IC5.K; no longer IC4.K
- net N$50: now also IC4.K; no longer IC3.K
- net N$51: now also IC8.B, R40.2, R41.2; no longer IC7.B, R35.2, R36.2
- net N$52: now also IC8.A, R42.2, R43.2; no longer IC7.A, R37.2, R38.2
- net N$53: now also IC8.!RE, IC8.DE, R37.2, R38.2; no longer IC7.!RE, IC7.DE, R32.2, R33.2
- net N$54: now also R42.1; no longer R37.1
- net N$55: now also R23.1; no longer R18.1
- net N$57: now also C10.2; no longer C9.2
- net N$58: now also BAT1.+, C21.2, IC3.VBAT; no longer IC8.CK, R12.1
- net N$59: now also R26.2, R27.2; no longer R20.2, R21.2
- net N$6: now also R10.1, R9.2; no longer R6.2, R7.1
- net N$61: now also R36.1; no longer R31.1
- net N$62: now also R39.1; no longer R34.1
- net N$63: now also R38.1; no longer R33.1
- net N$65: now also C12.2; no longer C11.2
- net N$66: now also C12.1; no longer C11.1
- net N$68: now also C26.2, IC6.IN+, R26.1; no longer C22.2, IC5.IN+, R20.1
- net N$69: now also C26.1, IC6.IN-, IC6.VBUS, R28.1; no longer C22.1, IC5.IN-, IC5.VBUS, R22.1
- net N$7: now also R11.2, R12.1; no longer R8.2, R9.1
- net N$70: now also IC3.!INT, R15.1, R18.2; no longer IC8.DI, R13.1
- net N$71: now also R29.2; no longer R23.2
- net N$72: now also C11.1, R7.2, R8.2; no longer C10.1, R4.2, R5.2
- net N$73: now also IC3.SCL, IC7.SCL, R20.2; no longer IC5.SCL, R29.2
- net N$77: now also C24.2, C25.2, IC6.VS; no longer C20.2, C21.2, IC5.VS
- net N$79: now also IC3.SDA, IC7.SDA, R19.2; no longer IC5.SDA, R28.2
- net N$8: now also R6.2; no longer R45.2
- net N$80: now also R41.1; no longer R36.1
- net N$85: now also R21.1; no longer R16.1
- net N$9: now also R16.2; no longer R13.2
- net UVCC: now also C9.2; no longer C8.2
- net VCC: now also C11.2, C15.2, C19.2, C20.2, C30.2, C33.2, IC3.VCC, IC7.A0, R18.1, R20.1, R22.1, R24.1, R25.1, R3.1, R34.1, R35.1, R4.2, R43.1, R7.1; no longer C10.2, C12.2, C26.2, C27.2, C29.1, C30.1, IC6.A0, IC7.VCC, IC8.!HOLD, IC8.!WP, R1.1, R15.1, R17.1, R23.1, R27.1, R28.1, R38.1, R4.1, R43.2, R47.1
Other:
- moved on the sheet: C10, C11, C12, C13, C14, C15, C16, C17, C18, C19, C20, C21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

Commit message: do
Parts:
- removed D4, D5: (no value), myparts:DIODE-SCHOTTKY
- removed Q1, Q2: (no value), myparts:N-MOSFET
- removed R44, R45, R46, R47: (no value), myparts:RESISTOR-0603
- added IC10, IC9: (no value), myparts:NUD3105-12-24-60
- SW3, SW4: device myparts:HK19F -> myparts:HFD2-L2
Connections:
- removed net N$36: Q1.G, R44.1, R45.2
- removed net N$37: D4.A, Q1.D, SW3.L2
- new net N$64: IC10.D_1, SW4.L1-
- new net N$82: IC10.D_2, SW4.L2-
- new net N$90: IC1.ADC5/PF5, IC9.G_2
- new net N$91: IC1.ADC4/PF4, IC9.G_1
- net GND: now also IC10.S_1, IC10.S_2, IC9.S_1, IC9.S_2; no longer Q1.S, Q2.S, R45.1, R47.1
- net N$24: now also IC1.ADC7/PF7, IC10.G_2; no longer IC1.ADC10/PD7, R46.2
- net N$26: now also IC9.D_1, SW3.L1-; no longer Q2.G, R46.1, R47.2
- net N$28: now also IC9.D_2, SW3.L2-; no longer D5.A, Q2.D, SW4.L2
- net N$32: now also IC1.PCINT4/ADC11/PB4; no longer IC1.PCINT5/ADC12/PB5
- net N$35: now also IC1.PCINT5/ADC12/PB5; no longer IC1.PCINT4/ADC11/PB4
- net N$38: now also IC1.ADC6/PF6, IC10.G_1; no longer IC1.ADC9/PD6, R44.2
- net VCC: now also SW3.L1+, SW3.L2+, SW4.L1+, SW4.L2+; no longer D4.K, D5.K, SW3.L1, SW4.L1
Other:
- moved on the sheet: C16, C17, C18, CON2, CON3, CON6, MOD1, R10, R11, R12, R13, R14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

Commit message: do
Other:
- moved on the sheet: SW1, SW2
Changed lines of the file:
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@@
 <attribute name="VALUE" x="20.32" y="-41.148" size="1.778" layer="96"/>
 </instance>
-<instance part="GND24" gate="1" x="132.08" y="78.74" smashed="yes" rot="R270">
-<attribute name="VALUE" x="129.032" y="81.28" size="1.778" layer="96" rot="R270"/>
+<instance part="GND24" gate="1" x="40.64" y="78.74" smashed="yes" rot="R270">
+<attribute name="VALUE" x="37.592" y="81.28" size="1.778" layer="96" rot="R270"/>
 </instance>
 <instance part="CON2" gate="G$1" x="68.58" y="7.62" smashed="yes">
@@
 <attribute name="VALUE" x="74.295" y="-86.995" size="1.778" layer="96"/>
 </instance>
-<instance part="SW1" gate="G$1" x="147.32" y="76.2" smashed="yes" rot="R180">
-<attribute name="NAME" x="144.526" y="72.644" size="1.778" layer="95" rot="R180" align="center-left"/>
-<attribute name="VALUE" x="144.526" y="70.866" size="1.778" layer="96" rot="R180" align="center-left"/>
-</instance>
-<instance part="GND69" gate="1" x="132.08" y="76.2" smashed="yes" rot="R270">
-<attribute name="VALUE" x="129.032" y="78.74" size="1.778" layer="96" rot="R270"/>
-</instance>
-<instance part="GND70" gate="1" x="149.86" y="76.2" smashed="yes" rot="R90">
-<attribute name="VALUE" x="152.908" y="73.66" size="1.778" layer="96" rot="R90"/>
-</instance>
-<instance part="SW2" gate="G$1" x="119.38" y="76.2" smashed="yes" rot="R180">
-<attribute name="NAME" x="116.586" y="72.644" size="1.778" layer="95" rot="R180" align="center-left"/>
-<attribute name="VALUE" x="116.586" y="70.866" size="1.778" layer="96" rot="R180" align="center-left"/>
-</instance>
-<instance part="GND71" gate="1" x="104.14" y="76.2" smashed="yes" rot="R270">
-<attribute name="VALUE" x="101.092" y="78.74" size="1.778" layer="96" rot="R270"/>
-</instance>
-<instance part="GND72" gate="1" x="121.92" y="76.2" smashed="yes" rot="R90">
-<attribute name="VALUE" x="124.968" y="73.66" size="1.778" layer="96" rot="R90"/>
+<instance part="SW1" gate="G$1" x="55.88" y="76.2" smashed="yes" rot="R180">
+<attribute name="NAME" x="53.086" y="72.644" size="1.778" layer="95" rot="R180" align="center-left"/>
+<attribute name="VALUE" x="53.086" y="70.866" size="1.778" layer="96" rot="R180" align="center-left"/>
+</instance>
+<instance part="GND69" gate="1" x="40.64" y="76.2" smashed="yes" rot="R270">
+<attribute name="VALUE" x="37.592" y="78.74" size="1.778" layer="96" rot="R270"/>
+</instance>
+<instance part="GND70" gate="1" x="58.42" y="76.2" smashed="yes" rot="R90">
+<attribute name="VALUE" x="61.468" y="73.66" size="1.778" layer="96" rot="R90"/>
+</instance>
+<instance part="SW2" gate="G$1" x="81.28" y="76.2" smashed="yes" rot="R180">
+<attribute name="NAME" x="78.486" y="72.644" size="1.778" layer="95" rot="R180" align="center-left"/>
+<attribute name="VALUE" x="78.486" y="70.866" size="1.778" layer="96" rot="R180" align="center-left"/>
+</instance>
+<instance part="GND71" gate="1" x="66.04" y="76.2" smashed="yes" rot="R270">
+<attribute name="VALUE" x="62.992" y="78.74" size="1.778" layer="96" rot="R270"/>
+</instance>
+<instance part="GND72" gate="1" x="83.82" y="76.2" smashed="yes" rot="R90">
+<attribute name="VALUE" x="86.868" y="73.66" size="1.778" layer="96" rot="R90"/>
 </instance>
 <instance part="SUP28" gate="G$1" x="-43.18" y="20.32" smashed="yes" rot="R180">
 <attribute name="VALUE" x="-41.275" y="18.415" size="1.778" layer="96" rot="R180"/>
 </instance>
-<instance part="GND13" gate="1" x="104.14" y="78.74" smashed="yes" rot="R270">
-<attribute name="VALUE" x="101.092" y="81.28" size="1.778" layer="96" rot="R270"/>
+<instance part="GND13" gate="1" x="66.04" y="78.74" smashed="yes" rot="R270">
+<attribute name="VALUE" x="62.992" y="81.28" size="1.778" layer="96" rot="R270"/>
 </instance>
 <instance part="C32" gate="G$1" x="-215.9" y="-121.92" smashed="yes" rot="R90">
@@
 <wire x1="-35.56" y1="12.7" x2="-35.56" y2="35.56" width="0.1524" layer="91"/>
 <wire x1="-35.56" y1="35.56" x2="-35.56" y2="50.8" width="0.1524" layer="91"/>
-<wire x1="-35.56" y1="50.8" x2="124.46" y2="50.8" width="0.1524" layer="91"/>
+<wire x1="-35.56" y1="50.8" x2="86.36" y2="50.8" width="0.1524" layer="91"/>
 <wire x1="-40.64" y1="35.56" x2="-35.56" y2="35.56" width="0.1524" layer="91"/>
 <junction x="-40.64" y="35.56"/>
 <junction x="-35.56" y="35.56"/>
-<wire x1="124.46" y1="50.8" x2="124.46" y2="78.74" width="0.1524" layer="91"/>
+<wire x1="86.36" y1="50.8" x2="86.36" y2="78.74" width="0.1524" layer="91"/>
 <pinref part="SW2" gate="G$1" pin="1"/>
-<wire x1="124.46" y1="78.74" x2="119.38" y2="78.74" width="0.1524" layer="91"/>
+<wire x1="86.36" y1="78.74" x2="81.28" y2="78.74" width="0.1524" layer="91"/>
 </segment>
 </net>
@@
 <wire x1="-25.4" y1="-40.64" x2="-25.4" y2="-48.26" width="0.1524" layer="91"/>
 <pinref part="SW1" gate="G$1" pin="1"/>
-<wire x1="147.32" y1="78.74" x2="152.4" y2="78.74" width="0.1524" layer="91"/>
-<wire x1="152.4" y1="78.74" x2="152.4" y2="48.26" width="0.1524" layer="91"/>
-<wire x1="152.4" y1="48.26" x2="60.96" y2="48.26" width="0.1524" layer="91"/>
-<wire x1="60.96" y1="48.26" x2="60.96" y2="-71.12" width="0.1524" layer="91"/>
+<wire x1="55.88" y1="78.74" x2="60.96" y2="78.74" width="0.1524" layer="91"/>
+<wire x1="60.96" y1="78.74" x2="60.96" y2="-71.12" width="0.1524" layer="91"/>
 <wire x1="60.96" y1="-71.12" x2="-30.48" y2="-71.12" width="0.1524" layer="91"/>
 <wire x1="-30.48" y1="-71.12" x2="-30.48" y2="-48.26" width="0.1524" layer="91"/>

Commit message: do
Connections:
- new net N$36: IC1.ADC0/PF0, R6.1
- net GND: no longer R6.1
- net N$1: now also IC1.ADC1/PF1; no longer IC1.ADC0/PF0
Changed lines of the file:
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@@
 <part name="R5" library="myparts" deviceset="RESISTOR-0603" device=""/>
 <part name="SUP7" library="myparts" deviceset="VCC" device=""/>
-<part name="GND25" library="myparts" deviceset="GND" device=""/>
 <part name="R38" library="myparts" deviceset="RESISTOR-0603" device=""/>
 <part name="R36" library="myparts" deviceset="RESISTOR-0603" device=""/>
@@
 <attribute name="VALUE" x="-41.275" y="73.025" size="1.778" layer="96" rot="R270"/>
 </instance>
-<instance part="GND25" gate="1" x="-73.66" y="73.66" smashed="yes" rot="R270">
-<attribute name="VALUE" x="-76.708" y="76.2" size="1.778" layer="96" rot="R270"/>
-</instance>
 <instance part="R38" gate="G$1" x="40.64" y="-109.22" smashed="yes">
 <attribute name="NAME" x="38.608" y="-108.204" size="1.778" layer="95" align="center-left"/>
@@
 <pinref part="C8" gate="G$1" pin="2"/>
 <pinref part="GND27" gate="1" pin="GND"/>
-</segment>
-<segment>
-<pinref part="R6" gate="G$1" pin="1"/>
-<pinref part="GND25" gate="1" pin="GND"/>
 </segment>
 <segment>
@@
 <pinref part="R1" gate="G$1" pin="1"/>
 <wire x1="-53.34" y1="7.62" x2="-55.88" y2="7.62" width="0.1524" layer="91"/>
-<wire x1="-55.88" y1="7.62" x2="-55.88" y2="58.42" width="0.1524" layer="91"/>
-<wire x1="-55.88" y1="58.42" x2="-27.94" y2="58.42" width="0.1524" layer="91"/>
-<wire x1="-27.94" y1="58.42" x2="-27.94" y2="68.58" width="0.1524" layer="91"/>
+<wire x1="-55.88" y1="7.62" x2="-55.88" y2="55.88" width="0.1524" layer="91"/>
+<wire x1="-55.88" y1="55.88" x2="-27.94" y2="55.88" width="0.1524" layer="91"/>
+<wire x1="-27.94" y1="55.88" x2="-27.94" y2="68.58" width="0.1524" layer="91"/>
 <pinref part="CON4" gate="G$1" pin="2"/>
 </segment>
@@
 <pinref part="R2" gate="G$1" pin="1"/>
 <wire x1="-53.34" y1="5.08" x2="-58.42" y2="5.08" width="0.1524" layer="91"/>
-<wire x1="-58.42" y1="5.08" x2="-58.42" y2="60.96" width="0.1524" layer="91"/>
-<wire x1="-58.42" y1="60.96" x2="-30.48" y2="60.96" width="0.1524" layer="91"/>
-<wire x1="-30.48" y1="60.96" x2="-30.48" y2="68.58" width="0.1524" layer="91"/>
+<wire x1="-58.42" y1="5.08" x2="-58.42" y2="58.42" width="0.1524" layer="91"/>
+<wire x1="-58.42" y1="58.42" x2="-30.48" y2="58.42" width="0.1524" layer="91"/>
+<wire x1="-30.48" y1="58.42" x2="-30.48" y2="68.58" width="0.1524" layer="91"/>
 <pinref part="CON4" gate="G$1" pin="3"/>
 </segment>
@@
 <pinref part="R5" gate="G$1" pin="1"/>
 <wire x1="-71.12" y1="63.5" x2="-71.12" y2="71.12" width="0.1524" layer="91"/>
-<pinref part="IC1" gate="G$1" pin="ADC0/PF0"/>
-<wire x1="-71.12" y1="63.5" x2="-5.08" y2="63.5" width="0.1524" layer="91"/>
-<wire x1="-5.08" y1="63.5" x2="-5.08" y2="35.56" width="0.1524" layer="91"/>
+<wire x1="-71.12" y1="63.5" x2="-2.54" y2="63.5" width="0.1524" layer="91"/>
+<pinref part="IC1" gate="G$1" pin="ADC1/PF1"/>
+<wire x1="-2.54" y1="63.5" x2="-2.54" y2="35.56" width="0.1524" layer="91"/>
 </segment>
 </net>
@@
 <wire x1="-327.66" y1="-106.68" x2="-327.66" y2="-86.36" width="0.1524" layer="91"/>
 <wire x1="-327.66" y1="-86.36" x2="-182.88" y2="-86.36" width="0.1524" layer="91"/>
-<wire x1="-182.88" y1="-86.36" x2="-182.88" y2="55.88" width="0.1524" layer="91"/>
-<wire x1="-25.4" y1="68.58" x2="-25.4" y2="55.88" width="0.1524" layer="91"/>
-<wire x1="-25.4" y1="55.88" x2="-182.88" y2="55.88" width="0.1524" layer="91"/>
+<wire x1="-182.88" y1="-86.36" x2="-182.88" y2="53.34" width="0.1524" layer="91"/>
+<wire x1="-25.4" y1="68.58" x2="-25.4" y2="53.34" width="0.1524" layer="91"/>
+<wire x1="-25.4" y1="53.34" x2="-182.88" y2="53.34" width="0.1524" layer="91"/>
 <pinref part="CON4" gate="G$1" pin="1"/>
 </segment>
@@
 </segment>
 </net>
+<net name="N$36" class="0">
+<segment>
+<pinref part="R6" gate="G$1" pin="1"/>
+<wire x1="-71.12" y1="73.66" x2="-73.66" y2="73.66" width="0.1524" layer="91"/>
+<wire x1="-73.66" y1="73.66" x2="-73.66" y2="60.96" width="0.1524" layer="91"/>
+<wire x1="-73.66" y1="60.96" x2="-5.08" y2="60.96" width="0.1524" layer="91"/>
+<pinref part="IC1" gate="G$1" pin="ADC0/PF0"/>
+<wire x1="-5.08" y1="60.96" x2="-5.08" y2="35.56" width="0.1524" layer="91"/>
+</segment>
+</net>

Commit message: do
Connections:
- net N$36: now also IC1.PB7/PCINT7; no longer IC1.ADC0/PF0
Changed lines of the file:
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@@
 <pinref part="R16" gate="G$1" pin="1"/>
 <wire x1="-127" y1="-109.22" x2="-129.54" y2="-109.22" width="0.1524" layer="91"/>
-<wire x1="-76.2" y1="-10.16" x2="-81.28" y2="-10.16" width="0.1524" layer="91"/>
-<wire x1="-81.28" y1="-10.16" x2="-81.28" y2="-88.9" width="0.1524" layer="91"/>
-<wire x1="-81.28" y1="-88.9" x2="-127" y2="-88.9" width="0.1524" layer="91"/>
+<wire x1="-76.2" y1="-10.16" x2="-83.82" y2="-10.16" width="0.1524" layer="91"/>
+<wire x1="-83.82" y1="-10.16" x2="-83.82" y2="-88.9" width="0.1524" layer="91"/>
+<wire x1="-83.82" y1="-88.9" x2="-127" y2="-88.9" width="0.1524" layer="91"/>
 <wire x1="-127" y1="-88.9" x2="-127" y2="-109.22" width="0.1524" layer="91"/>
 <junction x="-127" y="-109.22"/>
@@
 <pinref part="R17" gate="G$1" pin="1"/>
 <wire x1="-50.8" y1="-109.22" x2="-53.34" y2="-109.22" width="0.1524" layer="91"/>
-<wire x1="-76.2" y1="-12.7" x2="-78.74" y2="-12.7" width="0.1524" layer="91"/>
-<wire x1="-78.74" y1="-12.7" x2="-78.74" y2="-88.9" width="0.1524" layer="91"/>
-<wire x1="-78.74" y1="-88.9" x2="-50.8" y2="-88.9" width="0.1524" layer="91"/>
+<wire x1="-76.2" y1="-12.7" x2="-81.28" y2="-12.7" width="0.1524" layer="91"/>
+<wire x1="-81.28" y1="-12.7" x2="-81.28" y2="-88.9" width="0.1524" layer="91"/>
+<wire x1="-81.28" y1="-88.9" x2="-50.8" y2="-88.9" width="0.1524" layer="91"/>
 <wire x1="-50.8" y1="-88.9" x2="-50.8" y2="-109.22" width="0.1524" layer="91"/>
 <junction x="-50.8" y="-109.22"/>
@@
 <segment>
 <pinref part="R6" gate="G$1" pin="1"/>
-<wire x1="-71.12" y1="73.66" x2="-73.66" y2="73.66" width="0.1524" layer="91"/>
-<wire x1="-73.66" y1="73.66" x2="-73.66" y2="60.96" width="0.1524" layer="91"/>
-<wire x1="-73.66" y1="60.96" x2="-5.08" y2="60.96" width="0.1524" layer="91"/>
-<pinref part="IC1" gate="G$1" pin="ADC0/PF0"/>
-<wire x1="-5.08" y1="60.96" x2="-5.08" y2="35.56" width="0.1524" layer="91"/>
-</segment>
-</net>
+<wire x1="-71.12" y1="73.66" x2="-78.74" y2="73.66" width="0.1524" layer="91"/>
+<pinref part="IC1" gate="G$1" pin="PB7/PCINT7"/>
+<wire x1="-12.7" y1="-35.56" x2="-12.7" y2="-38.1" width="0.1524" layer="91"/>
+<wire x1="-12.7" y1="-38.1" x2="-78.74" y2="-38.1" width="0.1524" layer="91"/>
+<wire x1="-78.74" y1="-38.1" x2="-78.74" y2="73.66" width="0.1524" layer="91"/>
+</segment>
+</net>
